File: hardware/Li Charger.kicad_sch (KiCad schematic)
At the start: 31 parts, among them J1 USB_C_Receptacle_PowerOnly_6P, J2 Conn_01x02, U1 BQ24092DGQR, U2 LM3914V

Commit message: Schematic Value Update
Parts:
- R1: value R_Small -> 540
- R2: value R_Small -> 2k
Changed lines of the file:
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@@
 			)
 		)
-		(property "Value" "R_Small"
+		(property "Value" "2k"
 			(at 139.954 84.328 0)
 			(show_name no)
@@
 			)
 		)
-		(property "Value" "R_Small"
+		(property "Value" "540"
 			(at 132.08 74.93 0)
 			(show_name no)
